File: circuit.kicad_pcb (KiCad board)
At the start: 2 copper layers, 52 x 57.5 mm, 70 parts, among them J1 1725656, J2 CTX 3V3 GND TX, J3 CRX 3V3 GND RX, J4 PICO GP4/GP5 CAN, J5 2171750001, Q1 PMV100EPAR, U1 SN65HVD230DR, U2 AMS1117-3.3_C347222

Commit message: (karl) updates
Parts:
- TP41: value 3V3 -> +3.3V
- TP42: value 5V_USB -> +5VD
- TP43: value VIN12 -> +12V
- moved J3 37.7 mm to (156.6, 79.4), turned to -90 degrees
- moved TP43 34.9 mm to (141.6, 55.7)
- moved Q1 29.9 mm to (137.2, 49.1), turned to -90 degrees
- moved TP39 29.2 mm to (113.5, 42.5)
- moved TP40 29.2 mm to (113.5, 47.5)
- moved TP1 27.3 mm to (140.8, 42.5)
- moved J2 23.1 mm to (156.6, 75.3), turned to -90 degrees
- moved R3 22.1 mm to (152.7, 55.9)
- moved TP2 20.6 mm to (133.5, 42.5)
- moved D2 18.3 mm to (135.5, 55.1), turned to 180 degrees
- moved C5 17.6 mm to (155.5, 70.9), turned to 180 degrees
- moved U2 17.1 mm to (136.0, 61.8)
- moved U1 17.0 mm to (155.5, 62.9), turned to 0 degrees
- moved R1 16.5 mm to (135.3, 51.8), turned to 180 degrees
- moved C2 16.0 mm to (142.8, 63.3), turned to -90 degrees
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Routing:
- net CAN_RS: track 86.1 -> 4.19 mm, vias 2 -> 0
- net VIN12: track 75.5 -> 16.7 mm, vias 2 -> 0
- net VIN_RAW: track 51.2 -> 2.21 mm, vias 2 -> 0
- net CAN_RX: track 10.5 -> 50.5 mm
- net 3V3: track 93.4 -> 57.2 mm
- net 5V_USB: track 59.0 -> 28.6 mm, vias 3 -> 2
- net ACC12: track 26.1 -> 4.01 mm
- net BAT12: track 22.2 -> 4.05 mm
- net RP_GATE: track 17.2 -> 1.69 mm
- net CANL: track 32.2 -> 20.1 mm
- net TERM_SW: track 11.4 -> 2.04 mm, vias 2 -> 0
- net PWR_LED_A: track 10.7 -> 1.50 mm
- net GND: track 9.02 -> 0.00 mm, vias 5 -> 0
- net CC2: track 10.2 -> 4.82 mm
- net CC1: track 10.7 -> 6.32 mm, vias 2 -> 0
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
Commit message: progress
Parts:
- added D3: 15V, Library:SOD-123_L2.7-W1.6-LS3.7-RD, F.Cu at (141.5, 50.5)
- added D4: PESD5V0V1BB, Library:SOD-523_L1.2-W0.8-LS1.6-RD, F.Cu at (129.0, 82.5)
- added FB1: 600Ω@100MHz 1A, Resistor_SMD:R_0603_1608Metric, F.Cu at (130.5, 86.5)
- added JP3: PICO 3V3 ISO, Jumper:SolderJumper-2_P1.3mm_Open_RoundedPad1.0x1.5mm, F.Cu at (147.0, 43.0)
- D2: value SMBJ18A -> SMBJ15A; footprint Diode_SMD:D_SMB -> Library:SMB_L4.6-W3.6-LS5.3-RD
- J2, J3: footprint Connector_PinHeader_2.54mm:PinHeader_1x03_P2.54mm_Vertical -> Library:CONN-TH_705430002
- J4: footprint Connector_PinHeader_2.54mm:PinHeader_2x05_P2.54mm_Vertical -> Library:HDR-TH_10P-P2.54-V-M-R2-C5-S2.54
- R1: value 100kΩ -> 820Ω
- TP41: value +3.3V -> 3V3
- TP42: value +5VD -> 5V_USB
- TP43: value +12V -> VIN12
- moved J4 9.26 mm to (138.4, 76.2), turned to 180 degrees
- moved TP41 5.00 mm to (129.0, 66.0), turned to 180 degrees
Connections:
- J2 pad 1: 3V3 -> PICO_3V3
- J3 pad 1: 3V3 -> PICO_3V3
- J4 pad 10: (no net) -> unconnected-(J4-Pad10)
- J4 pad 3: 3V3 -> PICO_3V3
- J4 pad 7: (no net) -> unconnected-(J4-Pad7)
- J4 pad 8: (no net) -> unconnected-(J4-Pad8)
- J4 pad 9: (no net) -> unconnected-(J4-Pad9)
- J5 pad A9: 5V_USB -> VBUS
- J5 pad B9: 5V_USB -> VBUS
- JP1 pad 2: VIN_RAW -> unconnected-(JP1-C-Pad2)
- Q1 pad 3: VIN_RAW -> unconnected-(Q1-D-Pad3)
- R4 pad 2: TERM_SW -> CANL
- U1 pad 5: (no net) -> unconnected-(U1-VREF-Pad5)
Routing:
- net PICO_3V3: track 0.00 -> 89.3 mm, vias 0 -> 1
- net CAN_RX: track 50.5 -> 33.3 mm
- net 3V3: track 57.2 -> 71.9 mm
- net VBUS: track 0.00 -> 10.5 mm
- net GND: track 0.00 -> 9.67 mm
- net CAN_TX: track 37.5 -> 28.2 mm, vias 0 -> 1
- net VIN12: track 16.7 -> 25.5 mm
- net RP_GATE: track 1.69 -> 9.40 mm
- net 5V_USB: track 28.6 -> 35.6 mm
- net CANL: track 20.1 -> 24.1 mm
- net VIN_RAW: track 2.21 -> 0.00 mm
- net CAN_RS: track 4.19 -> 6.29 mm
- net CANH: track 20.8 -> 22.3 mm
Other:
- board text removed: "IMAGE HERE"
