File: circuit.kicad_pcb (KiCad board)
At the start: 2 copper layers, 52 x 57.5 mm, 74 parts, among them J1 1725656, J2 CTX 3V3 GND TX, J3 CRX 3V3 GND RX, J4 PICO GP4/GP5 CAN, J5 2171750001, Q1 PMV100EPAR, U1 SN65HVD230DR, U2 AMS1117-3.3_C347222

Commit message: more updates
Parts:
- removed J2: CTX 3V3 GND TX, Library:CONN-TH_705430002
- removed J3: CRX 3V3 GND RX, Library:CONN-TH_705430002
- removed JP2: TERM OPEN, Jumper:SolderJumper-2_P1.3mm_Open_RoundedPad1.0x1.5mm
- moved C1 34.4 mm to (178.8, 53.5)
- moved C3 31.4 mm to (178.8, 65.8)
- moved JP3 30.4 mm to (149.5, 73.2)
- moved TP41 29.7 mm to (157.5, 74.2), turned to 0 degrees
- moved C2 28.9 mm to (157.2, 88.2)
- moved D1 23.6 mm to (148.2, 88.7)
- moved TP1 19.8 mm to (128.8, 26.8)
- moved C5 19.7 mm to (166.8, 54.8)
- moved C4 19.7 mm to (166.8, 52.8)
- moved U2 19.5 mm to (154.8, 67.0)
- moved TP2 18.8 mm to (123.2, 26.8)
- moved JP1 18.6 mm to (126.2, 30.8)
- moved R2 17.7 mm to (155.2, 77.1)
- moved D2 14.1 mm to (148.4, 60.8)
- moved R1 11.9 mm to (141.4, 62.0)
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Routing:
- net PICO_3V3: track 89.3 -> 9.86 mm, vias 1 -> 0
- net 3V3: track 71.9 -> 47.9 mm
- net 5V_USB: track 35.6 -> 21.2 mm, vias 2 -> 0
- net CAN_RX: track 33.3 -> 21.4 mm, vias 0 -> 2
- net PWR_LED_A: track 1.75 -> 12.9 mm
- net CAN_TX: track 28.2 -> 17.2 mm, vias 1 -> 0
- net GND: track 9.67 -> 0.00 mm
- net VIN12: track 25.5 -> 33.6 mm, vias 0 -> 2
- net CANH: track 22.3 -> 14.7 mm
- net CANL: track 24.1 -> 17.8 mm
- net CC1: track 6.32 -> 12.3 mm, vias 0 -> 2
- net VBUS: track 10.5 -> 5.60 mm
- net BAT12: track 4.05 -> 0.00 mm
- net RP_GATE: track 9.40 -> 13.4 mm
- net ACC12: track 4.01 -> 0.00 mm
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
Commit message: pcb finishing
Parts:
- moved C1 45.4 mm to (133.5, 50.0), turned to 180 degrees
- moved C3 44.5 mm to (134.2, 66.2), turned to 180 degrees
- moved C5 33.6 mm to (134.3, 63.5)
- moved C4 33.6 mm to (134.3, 61.5)
- moved JP1 18.4 mm to (136.5, 46.0)
- moved TP1 18.4 mm to (139.0, 42.0)
- moved TP2 18.4 mm to (133.5, 42.0)
- moved R5 12.7 mm to (131.8, 85.3)
- moved D1 12.0 mm to (154.9, 78.7)
- moved D4 11.5 mm to (127.0, 83.5), turned to -90 degrees
- moved TP44 10.8 mm to (138.2, 84.3), turned to -90 degrees
- moved R6 10.5 mm to (133.6, 82.8)
- moved R1 10.00 mm to (132.5, 57.5)
- moved FB1 9.47 mm to (129.5, 77.7)
- moved C2 9.27 mm to (158.8, 79.1)
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Connections:
- J4 pad 10: unconnected-(J4-Pad10) -> (no net)
- J4 pad 7: unconnected-(J4-Pad7) -> (no net)
- J4 pad 8: unconnected-(J4-Pad8) -> (no net)
- J4 pad 9: unconnected-(J4-Pad9) -> (no net)
- JP1 pad 2: unconnected-(JP1-C-Pad2) -> VIN_RAW
- Q1 pad 3: unconnected-(Q1-D-Pad3) -> VIN_RAW
- U1 pad 5: unconnected-(U1-VREF-Pad5) -> (no net)
Routing:
- net VBUS: track 5.60 -> 23.4 mm, vias 0 -> 3
- net 3V3: track 47.9 -> 62.1 mm, vias 0 -> 2
- net VIN12: track 33.6 -> 46.4 mm
- net PWR_LED_A: track 12.9 -> 3.19 mm
- net CANL: track 17.8 -> 26.4 mm
- net CC1: track 12.3 -> 3.86 mm, vias 2 -> 0
- net VIN_RAW: track 0.00 -> 8.13 mm
- net CANH: track 14.7 -> 22.1 mm
- net ACC12: track 0.00 -> 4.41 mm
- net BAT12: track 0.00 -> 4.21 mm
- net CAN_RS: track 4.90 -> 8.68 mm
- net PICO_3V3: track 9.86 -> 12.8 mm
- net 5V_USB: track 21.2 -> 18.8 mm
- net CAN_TX: track 17.2 -> 19.1 mm
- net CAN_RX: track 21.4 -> 19.6 mm
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
Commit message: SILKSCREEN
Parts:
- added G***: LOGO, LOGO, F.Cu at (151.4, 93.5)
- added G***: LOGO, LOGO, F.Cu at (147.8, 86.4)
- added G***: LOGO, LOGO, B.Cu at (145.3, 57.4)
- added G***: LOGO, LOGO, B.Cu at (154.4, 89.9)
Other:
- outline, holes or cut-outs redrawn
- board text added: "J4 PICO HEADER pin 1 CAN_TX GP4 pin 2 GND pin 3 3V3 pin 4 CAN_RX GP5 pin 5 5V_USB"
- board text added: "MAZZY"
- board text added: "Mazzy Mini v1.0"
- board text added: "v1.0"
