File: circuit.kicad_sch (KiCad schematic)
At the start: 71 parts, among them J1 1725656, J4 PICO GP4/GP5 CAN, J5 2171750001, Q1 PMV100EPAR, U1 SN65HVD230DR, U2 AMS1117-3.3_C347222

Commit message: quick updates w/ new review things
Parts:
- R1: value 820Ω -> 10kΩ
